File: h_bridge.kicad_sch (KiCad schematic)
At the start: 33 parts, among them U3 INA180B3, U4 INA180B3, U5 INA180B3

Commit message: Correct current sense amplifier polarity and add decoupling capacitors
Parts:
- added C11, C12, C8: 100n, symbol Device:C
Connections:
- net +3.3V: now also C11.1, C12.1, C8.1
- net A: now also U3.3 (-); no longer U3.1 (+)
- net B: now also U4.3 (-); no longer U4.1 (+)
- net C: now also U5.3 (-); no longer U5.1 (+)
- net GND: now also C11.2, C12.2, C8.2
- net at A_H.3 (S), A_H.4 (D), A_L.2 (D)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: now also U3.1 (+); no longer U3.3 (-)
- net at C_H.3 (S), C_H.4 (D), C_L.2 (D)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: now also U5.1 (+); no longer U5.3 (-)
- net at B_H.3 (S), B_H.4 (D), B_L.2 (D)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: now also U4.1 (+); no longer U4.3 (-)
Other:
- moved on the sheet: U3, U4, U5
